File: motherboard.kicad_pcb (KiCad board)
At the start: 2 copper layers, 194.3 x 174 mm, 99 parts, among them J1 Conn_02x26_Odd_Even, J10 Conn_01x02, J2 Conn_02x24_Odd_Even, J3 Conn_02x24_Odd_Even, J4 Conn_02x24_Odd_Even, J5 Conn_02x24_Odd_Even, J6 Conn_02x08_Odd_Even, J7 Conn_01x03, J8 Barrel_Jack_Switch, J9 Conn_01x02, U1 68000D, U10 28C256, U11 74LS27, U12 74LS27, U13 74LS27, U14 74LS245, U15 74LS245, U16 28C256, U17 74LS08, U18 74LS08, U19 74LS08, U2 74LS02, U20 74LS245, U21 74LS245, U22 74LS05, U23 74LS138, U24 74LS245, U25 74LS245, U26 74HC164, U27 LM555, U28 L7805, U3 74LS00, U4 74LS32, U5 74LS245, U6 74LS245, U7 74LS04, U8 74LS10, U9 74LS10, X1 CXO_DIP8

Commit message: HC, HCT fix. Gerber archive removed. Scheme pdf added.
Parts:
- U11, U12, U13: value 74LS27 -> 74HC27
- U14, U15, U20, U21, U24, U25, U5, U6: value 74LS245 -> 74HC245
- U17, U18, U19: value 74LS08 -> 74HC08
- U2: value 74LS02 -> 74HC02
- U22: value 74LS05 -> 74HC05
- U23: value 74LS138 -> 74HC138
- U3: value 74LS00 -> 74HC00
- U4: value 74LS32 -> 74HC32
- U7: value 74LS04 -> 74HC04
- U8, U9: value 74LS10 -> 74HC10
