File: motherboard.kicad_pcb (KiCad board)
At the start: 2 copper layers, 194.3 x 174 mm, 99 parts, among them J1 Conn_02x26_Odd_Even, J10 Conn_01x02, J2 Conn_02x24_Odd_Even, J3 Conn_02x24_Odd_Even, J4 Conn_02x24_Odd_Even, J5 Conn_02x24_Odd_Even, J6 Conn_02x08_Odd_Even, J7 Conn_01x03, J8 Barrel_Jack_Switch, J9 Conn_01x02, U1 68000D, U10 28C256, U11 74HC27, U12 74HC27, U13 74HC27, U14 74HC245, U15 74HC245, U16 28C256, U17 74HC08, U18 74HC08, U19 74HC08, U2 74HC02, U20 74HC245, U21 74HC245, U22 74HC05, U23 74HC138, U24 74HC245, U25 74HC245, U26 74HC164, U27 LM555, U28 L7805, U3 74HC00, U4 74HC32, U5 74HC245, U6 74HC245, U7 74HC04, U8 74HC10, U9 74HC10, X1 CXO_DIP8

Commit message: 555 timer update
Parts:
- U27: value LM555 -> NE555P

Commit message: Gerber update
Other:
- rule pad_to_mask_clearance: 0.051 -> 0
Changed lines of the file:
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@@
     (pad_size 1.524 1.524)
     (pad_drill 0.762)
-    (pad_to_mask_clearance 0.051)
-    (solder_mask_min_width 0.25)
+    (pad_to_mask_clearance 0)
     (aux_axis_origin 0 0)
     (visible_elements FFFFFF7F)
     (pcbplotparams
-      (layerselection 0x010fc_ffffffff)
+      (layerselection 0x010f0_ffffffff)
       (usegerberextensions false)
-      (usegerberattributes false)
-      (usegerberadvancedattributes false)
+      (usegerberattributes true)
+      (usegerberadvancedattributes true)
       (creategerberjobfile false)
       (excludeedgelayer true)
@@
     (add_net "Net-(D1-Pad2)")
     (add_net "Net-(D2-Pad2)")
-    (add_net "Net-(HOLE1-Pad1)")
-    (add_net "Net-(HOLE2-Pad1)")
-    (add_net "Net-(HOLE3-Pad1)")
-    (add_net "Net-(HOLE4-Pad1)")
-    (add_net "Net-(J1-Pad24)")
-    (add_net "Net-(J1-Pad49)")
-    (add_net "Net-(J1-Pad51)")
     (add_net "Net-(J10-Pad1)")
-    (add_net "Net-(J2-Pad20)")
-    (add_net "Net-(J3-Pad20)")
-    (add_net "Net-(J4-Pad20)")
-    (add_net "Net-(J5-Pad20)")
     (add_net "Net-(J6-Pad1)")
     (add_net "Net-(J6-Pad11)")
@@
     (add_net "Net-(J7-Pad1)")
     (add_net "Net-(J7-Pad3)")
-    (add_net "Net-(J8-Pad3)")
-    (add_net "Net-(RN2-Pad4)")
-    (add_net "Net-(RN2-Pad5)")
-    (add_net "Net-(RN4-Pad6)")
-    (add_net "Net-(RN4-Pad7)")
-    (add_net "Net-(RN4-Pad8)")
-    (add_net "Net-(RN4-Pad9)")
-    (add_net "Net-(U1-Pad11)")
-    (add_net "Net-(U1-Pad19)")
-    (add_net "Net-(U1-Pad20)")
     (add_net "Net-(U11-Pad12)")
     (add_net "Net-(U11-Pad6)")
@@
     (add_net "Net-(U19-Pad1)")
     (add_net "Net-(U19-Pad13)")
-    (add_net "Net-(U2-Pad13)")
     (add_net "Net-(U2-Pad2)")
     (add_net "Net-(U2-Pad3)")
     (add_net "Net-(U22-Pad1)")
-    (add_net "Net-(U22-Pad10)")
-    (add_net "Net-(U22-Pad12)")
     (add_net "Net-(U22-Pad5)")
-    (add_net "Net-(U24-Pad15)")
     (add_net "Net-(U3-Pad1)")
     (add_net "Net-(U3-Pad12)")
-    (add_net "Net-(U5-Pad11)")
-    (add_net "Net-(X1-Pad1)")
     (add_net RESV_ADDR)
     (add_net ROM_DTACK)

Commit message: Footrpint fix
Connections:
- HOLE1 pad 1: (no net) -> Net-(HOLE1-Pad1)
- HOLE2 pad 1: (no net) -> Net-(HOLE2-Pad1)
- HOLE3 pad 1: (no net) -> Net-(HOLE3-Pad1)
- HOLE4 pad 1: (no net) -> Net-(HOLE4-Pad1)
- J1 pad 24: (no net) -> Net-(J1-Pad24)
- J1 pad 49: (no net) -> Net-(J1-Pad49)
- J1 pad 51: (no net) -> Net-(J1-Pad51)
- J2 pad 20: (no net) -> Net-(J2-Pad20)
- J3 pad 20: (no net) -> Net-(J3-Pad20)
- J4 pad 20: (no net) -> Net-(J4-Pad20)
- J5 pad 20: (no net) -> Net-(J5-Pad20)
- J8 pad 3: (no net) -> Net-(J8-Pad3)
- RN2 pad 4: (no net) -> Net-(RN2-Pad4)
- RN2 pad 5: (no net) -> Net-(RN2-Pad5)
- RN4 pad 6: (no net) -> Net-(RN4-Pad6)
- RN4 pad 7: (no net) -> Net-(RN4-Pad7)
- RN4 pad 8: (no net) -> Net-(RN4-Pad8)
- RN4 pad 9: (no net) -> Net-(RN4-Pad9)
- U1 pad 11: (no net) -> Net-(U1-Pad11)
- U1 pad 19: (no net) -> Net-(U1-Pad19)
- U1 pad 20: (no net) -> Net-(U1-Pad20)
- U2 pad 13: (no net) -> Net-(U2-Pad13)
- U22 pad 10: (no net) -> Net-(U22-Pad10)
- U22 pad 12: (no net) -> Net-(U22-Pad12)
- U24 pad 15: (no net) -> Net-(U24-Pad15)
- U5 pad 11: (no net) -> Net-(U5-Pad11)
- X1 pad 1: (no net) -> Net-(X1-Pad1)

Commit message: 74HCT245 and bypass capacitors fix
Parts:
- U14, U15, U20, U24, U5, U6: value 74HC245 -> 74HCT245
