File: motherboard.sch (KiCad schematic (older format))
At the start: 99 parts, among them J1 Conn_02x26_Odd_Even, J10 Conn_01x02, J2 Conn_02x24_Odd_Even, J3 Conn_02x24_Odd_Even, J4 Conn_02x24_Odd_Even, J5 Conn_02x24_Odd_Even, J6 Conn_02x08_Odd_Even, J7 Conn_01x03, J8 Barrel_Jack_Switch, J9 Conn_01x02, U1 68000D, U10 28C256, U11 74HC27, U12 74HC27, U13 74HC27, U14 74HC245, U15 74HC245, U16 28C256, U17 74HC08, U18 74HC08, U19 74HC08, U2 74HC02, U20 74HC245, U21 74HC245, U22 74HC05, U23 74HC138, U24 74HC245, U25 74HC245, U26 74HC164, U27 LM555, U28 L7805, U3 74HC00, U4 74HC32, U5 74HC245, U6 74HC245, U7 74HC04, U8 74HC10, U9 74HC10, X1 CXO_DIP8

Commit message: Description added
Other:
- note added: "BUS BUFFERS"
- note added: "BYTE READ"
- note added: "CAPACITORS"
- note added: "CLOCK"
- note added: "DEVICE SELECT"
- note added: "DTACK"
- note added: "HOLES"
- note added: "IRQ"
- note added: "MEM SELECT"
- note added: "PROCESSOR"
- note added: "PULL-UP RESISTORS"
- note added: "PWR CIRCUIT"
- note added: "PWR LED\n"
- note added: "RAM SLOT\nDEVICE SLOTS\n& etc"
- note added: "READ&WRITE"
- note added: "RESET"
- note added: "RESET DECODER"
- note added: "ROM CHIPS"
- note added: "ROM DECODER"
- note added: "ROM DTACK"
- note added: "ROM RQ"
- note added: "STATE DECODER"
- moved on the sheet: D2, HOLE1, HOLE2, HOLE3, HOLE4, J6, R10, U10, U13B, U13C, U16, U17A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

Commit message: 555 timer update
Parts:
- removed U27: LM555, Package_DIP:DIP-8_W7.62mm_Socket, symbol motherboard-rescue:LM555-Timer
- added U27: NE555P, Package_DIP:DIP-8_W7.62mm_Socket, symbol Timer:NE555P
Connections:
- net GND: now also U27.1 (GND)
- net VCC: now also U27.4 (R), U27.8 (VCC)
- net at C34.1, R6.2: now also U27.2 (TR)
- net at U22.1, U22.3: now also U27.3 (Q)
- net at C35.1: now also U27.5 (CV)
- net at C37.1, R9.2: now also U27.6 (THR), U27.7 (DIS)
Changed lines of the file:
@@
 $EndComp
 $Comp
-L motherboard-rescue:LM555-Timer U27
-U 1 1 5F41053C
-P 19700 9050
-F 0 "U27" H 19700 9631 50  0000 C CNN
-F 1 "LM555" H 19700 9540 50  0000 C CNN
-F 2 "Package_DIP:DIP-8_W7.62mm_Socket" H 19700 9050 50  0001 C CNN
-F 3 "http://www.ti.com/lit/ds/symlink/lm555.pdf" H 19700 9050 50  0001 C CNN
-	1    19700 9050
-	1    0    0    -1
-$EndComp
-$Comp
 L power:VCC #PWR073
 U 1 1 5FE911B5
@@
 Text Notes 10500 5000 0    100  ~ 20
 BUS BUFFERS
+$Comp
+L Timer:NE555P U27
+U 1 1 5FFCEDA1
+P 19700 9050
+F 0 "U27" H 19700 9631 50  0000 C CNN
+F 1 "NE555P" H 19700 9540 50  0000 C CNN
+F 2 "Package_DIP:DIP-8_W7.62mm_Socket" H 20350 8650 50  0001 C CNN
+F 3 "http://www.ti.com/lit/ds/symlink/ne555.pdf" H 20550 8650 50  0001 C CNN
+	1    19700 9050
+	1    0    0    -1
+$EndComp
 $EndSCHEMATC

Commit message: Footrpint fix
Parts:
- HOLE1, HOLE2, HOLE3, HOLE4: footprint plugins:HOLE_SUEN -> footprints:HOLE_SUEN
Changed lines of the file:
@@
 F 0 "HOLE1" H 21180 13492 50  0000 L CNN
 F 1 "Conn_01x01" H 21180 13401 50  0000 L CNN
-F 2 "plugins:HOLE_SUEN" H 21100 13450 50  0001 C CNN
+F 2 "footprints:HOLE_SUEN" H 21100 13450 50  0001 C CNN
 F 3 "~" H 21100 13450 50  0001 C CNN
 	1    21100 13450
@@
 F 0 "HOLE2" H 21180 13692 50  0000 L CNN
 F 1 "Conn_01x01" H 21180 13601 50  0000 L CNN
-F 2 "plugins:HOLE_SUEN" H 21100 13650 50  0001 C CNN
+F 2 "footprints:HOLE_SUEN" H 21100 13650 50  0001 C CNN
 F 3 "~" H 21100 13650 50  0001 C CNN
 	1    21100 13650
@@
 F 0 "HOLE3" H 21180 13892 50  0000 L CNN
 F 1 "Conn_01x01" H 21180 13801 50  0000 L CNN
-F 2 "plugins:HOLE_SUEN" H 21100 13850 50  0001 C CNN
+F 2 "footprints:HOLE_SUEN" H 21100 13850 50  0001 C CNN
 F 3 "~" H 21100 13850 50  0001 C CNN
 	1    21100 13850
@@
 F 0 "HOLE4" H 21180 14092 50  0000 L CNN
 F 1 "Conn_01x01" H 21180 14001 50  0000 L CNN
-F 2 "plugins:HOLE_SUEN" H 21100 14050 50  0001 C CNN
+F 2 "footprints:HOLE_SUEN" H 21100 14050 50  0001 C CNN
 F 3 "~" H 21100 14050 50  0001 C CNN
 	1    21100 14050

Commit message: More trash deleted, .gitignore added
Parts:
- HOLE1, HOLE2, HOLE3, HOLE4: footprint footprints:HOLE_SUEN -> footprints:Hole
Changed lines of the file:
@@
 F 0 "HOLE1" H 21180 13492 50  0000 L CNN
 F 1 "Conn_01x01" H 21180 13401 50  0000 L CNN
-F 2 "footprints:HOLE_SUEN" H 21100 13450 50  0001 C CNN
+F 2 "footprints:Hole" H 21100 13450 50  0001 C CNN
 F 3 "~" H 21100 13450 50  0001 C CNN
 	1    21100 13450
@@
 F 0 "HOLE2" H 21180 13692 50  0000 L CNN
 F 1 "Conn_01x01" H 21180 13601 50  0000 L CNN
-F 2 "footprints:HOLE_SUEN" H 21100 13650 50  0001 C CNN
+F 2 "footprints:Hole" H 21100 13650 50  0001 C CNN
 F 3 "~" H 21100 13650 50  0001 C CNN
 	1    21100 13650
@@
 F 0 "HOLE3" H 21180 13892 50  0000 L CNN
 F 1 "Conn_01x01" H 21180 13801 50  0000 L CNN
-F 2 "footprints:HOLE_SUEN" H 21100 13850 50  0001 C CNN
+F 2 "footprints:Hole" H 21100 13850 50  0001 C CNN
 F 3 "~" H 21100 13850 50  0001 C CNN
 	1    21100 13850
@@
 F 0 "HOLE4" H 21180 14092 50  0000 L CNN
 F 1 "Conn_01x01" H 21180 14001 50  0000 L CNN
-F 2 "footprints:HOLE_SUEN" H 21100 14050 50  0001 C CNN
+F 2 "footprints:Hole" H 21100 14050 50  0001 C CNN
 F 3 "~" H 21100 14050 50  0001 C CNN
 	1    21100 14050

Commit message: 74HCT245 and bypass capacitors fix
Parts:
- U14, U15, U20, U24, U5, U6: value 74HC245 -> 74HCT245
Other:
- note added: "BYPASS CAPACITORS"
- note removed: "CAPACITORS"
Changed lines of the file:
@@
-$EndComp
-$Comp
-L 74xx:74LS245 U5
-U 1 1 5F549BD8
-P 4450 1650
-F 0 "U5" H 4450 2631 50  0000 C CNN
-F 1 "74HC245" H 4450 2540 50  0000 C CNN
-F 2 "Package_DIP:DIP-20_W7.62mm_Socket" H 4450 1650 50  0001 C CNN
-F 3 "http://www.ti.com/lit/gpn/sn74LS245" H 4450 1650 50  0001 C CNN
-	1    4450 1650
-	1    0    0    -1
-$EndComp
-$Comp
-L 74xx:74LS245 U6
-U 1 1 5F563258
-P 4450 3900
-F 0 "U6" H 4450 4881 50  0000 C CNN
-F 1 "74HC245" H 4450 4790 50  0000 C CNN
-F 2 "Package_DIP:DIP-20_W7.62mm_Socket" H 4450 3900 50  0001 C CNN
-F 3 "http://www.ti.com/lit/gpn/sn74LS245" H 4450 3900 50  0001 C CNN
-	1    4450 3900
-	1    0    0    -1
-$EndComp
-$Comp
-L 74xx:74LS245 U14
-U 1 1 5F55E7F0
-P 6200 1650
-F 0 "U14" H 6200 2631 50  0000 C CNN
-F 1 "74HC245" H 6200 2540 50  0000 C CNN
-F 2 "Package_DIP:DIP-20_W7.62mm_Socket" H 6200 1650 50  0001 C CNN
-F 3 "http://www.ti.com/lit/gpn/sn74LS245" H 6200 1650 50  0001 C CNN
-	1    6200 1650
-	1    0    0    -1
-$EndComp
-$Comp
-L 74xx:74LS245 U15
-U 1 1 5F567FE9
-P 6300 3900
-F 0 "U15" H 6300 4881 50  0000 C CNN
-F 1 "74HC245" H 6300 4790 50  0000 C CNN
-F 2 "Package_DIP:DIP-20_W7.62mm_Socket" H 6300 3900 50  0001 C CNN
-F 3 "http://www.ti.com/lit/gpn/sn74LS245" H 6300 3900 50  0001 C CNN
-	1    6300 3900
-	1    0    0    -1
-$EndComp
-$Comp
-L 74xx:74LS245 U20
-U 1 1 5F55EE3D
-P 8000 1650
-F 0 "U20" H 8000 2631 50  0000 C CNN
-F 1 "74HC245" H 8000 2540 50  0000 C CNN
-F 2 "Package_DIP:DIP-20_W7.62mm_Socket" H 8000 1650 50  0001 C CNN
-F 3 "http://www.ti.com/lit/gpn/sn74LS245" H 8000 1650 50  0001 C CNN
-	1    8000 1650
-	1    0    0    -1
-$EndComp
-$Comp
-L 74xx:74LS245 U21
-U 1 1 5F568CC7
-P 8200 3900
-F 0 "U21" H 8200 4881 50  0000 C CNN
-F 1 "74HC245" H 8200 4790 50  0000 C CNN
-F 2 "Package_DIP:DIP-20_W7.62mm_Socket" H 8200 3900 50  0001 C CNN
-F 3 "http://www.ti.com/lit/gpn/sn74LS245" H 8200 3900 50  0001 C CNN
-	1    8200 3900
-	1    0    0    -1
-$EndComp
-$Comp
-L 74xx:74LS245 U24
-U 1 1 5F561142
-P 10250 1650
-F 0 "U24" H 10250 2631 50  0000 C CNN
-F 1 "74HC245" H 10250 2540 50  0000 C CNN
-F 2 "Package_DIP:DIP-20_W7.62mm_Socket" H 10250 1650 50  0001 C CNN
-F 3 "http://www.ti.com/lit/gpn/sn74LS245" H 10250 1650 50  0001 C CNN
-	1    10250 1650
-	1    0    0    -1
-$EndComp
-$Comp
-L 74xx:74LS245 U25
-U 1 1 5F569753
-P 10250 3900
-F 0 "U25" H 10250 4881 50  0000 C CNN
-F 1 "74HC245" H 10250 4790 50  0000 C CNN
-F 2 "Package_DIP:DIP-20_W7.62mm_Socket" H 10250 3900 50  0001 C CNN
-F 3 "http://www.ti.com/lit/gpn/sn74LS245" H 10250 3900 50  0001 C CNN
-	1    10250 3900
-	1    0    0    -1
 $EndComp
 $Comp
@@
 Text Notes 21450 13050 0    100  ~ 20
 HOLES
-Text Notes 17100 11200 0    100  ~ 20
-CAPACITORS
+Text Notes 16450 11200 0    100  ~ 20
+BYPASS CAPACITORS
 Text Notes 17350 6000 0    100  ~ 20
 IRQ
@@
 	1    0    0    -1
 $EndComp
+$Comp
+L 74xx:74LS245 U21
+U 1 1 5F568CC7
+P 8200 3900
+F 0 "U21" H 8200 4881 50  0000 C CNN
+F 1 "74HC245" H 8200 4790 50  0000 C CNN
+F 2 "Package_DIP:DIP-20_W7.62mm_Socket" H 8200 3900 50  0001 C CNN
+F 3 "http://www.ti.com/lit/gpn/sn74LS245" H 8200 3900 50  0001 C CNN
+	1    8200 3900
+	1    0    0    -1
+$EndComp
+$Comp
+L 74xx:74LS245 U25
+U 1 1 5F569753
+P 10250 3900
+F 0 "U25" H 10250 4881 50  0000 C CNN
+F 1 "74HC245" H 10250 4790 50  0000 C CNN
+F 2 "Package_DIP:DIP-20_W7.62mm_Socket" H 10250 3900 50  0001 C CNN
+F 3 "http://www.ti.com/lit/gpn/sn74LS245" H 10250 3900 50  0001 C CNN
+	1    10250 3900
+	1    0    0    -1
+$EndComp
+$Comp
+L 74xx:74LS245 U5
+U 1 1 5F549BD8
+P 4450 1650
+F 0 "U5" H 4450 2631 50  0000 C CNN
+F 1 "74HCT245" H 4450 2540 50  0000 C CNN
+F 2 "Package_DIP:DIP-20_W7.62mm_Socket" H 4450 1650 50  0001 C CNN
+F 3 "http://www.ti.com/lit/gpn/sn74LS245" H 4450 1650 50  0001 C CNN
+	1    4450 1650
+	1    0    0    -1
+$EndComp
+$Comp
+L 74xx:74LS245 U14
+U 1 1 5F55E7F0
+P 6200 1650
+F 0 "U14" H 6200 2631 50  0000 C CNN
+F 1 "74HCT245" H 6200 2540 50  0000 C CNN
+F 2 "Package_DIP:DIP-20_W7.62mm_Socket" H 6200 1650 50  0001 C CNN
+F 3 "http://www.ti.com/lit/gpn/sn74LS245" H 6200 1650 50  0001 C CNN
+	1    6200 1650
+	1    0    0    -1
+$EndComp
+$Comp
+L 74xx:74LS245 U20
+U 1 1 5F55EE3D
+P 8000 1650
+F 0 "U20" H 8000 2631 50  0000 C CNN
+F 1 "74HCT245" H 8000 2540 50  0000 C CNN
+F 2 "Package_DIP:DIP-20_W7.62mm_Socket" H 8000 1650 50  0001 C CNN
+F 3 "http://www.ti.com/lit/gpn/sn74LS245" H 8000 1650 50  0001 C CNN
+	1    8000 1650
+	1    0    0    -1
+$EndComp
+$Comp
+L 74xx:74LS245 U24
+U 1 1 5F561142
+P 10250 1650
+F 0 "U24" H 10250 2631 50  0000 C CNN
+F 1 "74HCT245" H 10250 2540 50  0000 C CNN
+F 2 "Package_DIP:DIP-20_W7.62mm_Socket" H 10250 1650 50  0001 C CNN
+F 3 "http://www.ti.com/lit/gpn/sn74LS245" H 10250 1650 50  0001 C CNN
+	1    10250 1650
+	1    0    0    -1
+$EndComp
+$Comp
+L 74xx:74LS245 U6
+U 1 1 5F563258
+P 4450 3900
+F 0 "U6" H 4450 4881 50  0000 C CNN
+F 1 "74HCT245" H 4450 4790 50  0000 C CNN
+F 2 "Package_DIP:DIP-20_W7.62mm_Socket" H 4450 3900 50  0001 C CNN
+F 3 "http://www.ti.com/lit/gpn/sn74LS245" H 4450 3900 50  0001 C CNN
+	1    4450 3900
+	1    0    0    -1
+$EndComp
+$Comp
+L 74xx:74LS245 U15
+U 1 1 5F567FE9
+P 6300 3900
+F 0 "U15" H 6300 4881 50  0000 C CNN
+F 1 "74HCT245" H 6300 4790 50  0000 C CNN
+F 2 "Package_DIP:DIP-20_W7.62mm_Socket" H 6300 3900 50  0001 C CNN
+F 3 "http://www.ti.com/lit/gpn/sn74LS245" H 6300 3900 50  0001 C CNN
+	1    6300 3900
+	1    0    0    -1
+$EndComp
